File: RB3202/hardware/SchoolBoard.brd (EAGLE design)
At the start: 101.6 x 61 mm, 83 parts, among them Q1 AO3401ASOP-8_EP_5.0X5.0X1.27P, Q3 AO3401ASOP-8_EP_5.0X5.0X1.27P, SW0 TL3342F160QG/TR, SW1 TL3342F160QG/TR, SW2 TL3342F160QG/TR, SW3 TL3342F160QG/TR, U1 MPU-6050, X1 POWER_IN, X2 POWER_IN, X4 POWER_IN

Commit message: kompas_navic
Parts:
- added C18: 220nf, rcl_upravena:C0402
- added C19: 4.7uf, rcl_upravena:C0805
- added C20, C21: 100nf, rcl_upravena:C0402P
- added IC3: QMC5883L-TR, QMC5883L-TR:QMC5882L-TR
- added JP11: (no value), pinhead:1X01
- C23: device resistor:C0603 -> resistor:C0402
- moved R23 3.69 mm to (4.32, 13.6)
- moved R22 3.68 mm to (5.74, 13.6)
- moved C23 0.25 mm to (74.2, 32.5)
Connections:
- new net IO10_NC2: IC3.6
- new net IO9_NC3: IC3.5
- new net IO9_NC6: IC3.14
- new net IO9_NC7: IC3.3
- new net IO9_NC8: IC3.7
- new net N$60: C18.1, IC3.12
- new net N$62: C18.2, IC3.8
- new net N$66: C19.1, IC3.10
- new net QMC5883-INTERRUPT: IC3.15, JP11.1
- net +3V3: now also C20.1, C21.1, IC3.13, IC3.2, IC3.4
- net GND: now also C19.2, C20.2, C21.2, IC3.11, IC3.9
- net SCL: now also IC3.1
- net SDA: now also IC3.16
Routing:
- net SDA: track 92.5 -> 122.3 mm
- net SCL: track 93.1 -> 116.5 mm
- net +3V3: track 136.8 -> 158.2 mm
- net N$62: track 0.00 -> 7.61 mm
- net N$60: track 0.00 -> 4.10 mm
- net VCC: track 81.3 -> 84.6 mm
- net QMC5883-INTERRUPT: track 0.00 -> 2.03 mm
- net N$66: track 0.00 -> 1.81 mm
Other:
- board text added: "+"
- board text added: "-"
- board text added: "1"
- board text added: "21"
- board text added: "25"
- board text added: "26"
- board text added: "27"
- board text added: "3"
- board text added: "35"
- board text added: "36"
- board text added: "39"
- board text added: "3V3"
- board text added: "5V"
- board text added: "A"
- board text added: "B"
- board text added: "GPIO"
- board text added: "I2C"
- board text added: "JESPER RB3202S_V1.0"
- board text added: "MPU-interupt"
- board text added: "QMC-interupt"
- board text added: "SCL"
- board text added: "SDA"
