File: RB3202/hardware/SchoolBoard.sch (EAGLE design)
At the start: 93 parts, among them Q1 AO3401ASOP-8_EP_5.0X5.0X1.27P, Q3 AO3401ASOP-8_EP_5.0X5.0X1.27P, SW0 TL3342F160QG/TR, SW1 TL3342F160QG/TR, SW2 TL3342F160QG/TR, SW3 TL3342F160QG/TR, U1 MPU-6050, X1 POWER_IN, X2 POWER_IN, X4 POWER_IN

Commit message: kompas_navic
Parts:
- added C18: 220nf, rcl_upravena:C-EUC0402
- added C19: 4.7uf, rcl_upravena:C-EUC0805
- added C20, C21: 100nf, rcl_upravena:C-EU
- added IC3: QMC5883L-TR, QMC5883L-TR:QMC5883L-TR
- added JP11: (no value), pinhead:PINHD-1X1
- added NC10, NC11, NC12, NC15, NC9: NC, NC:NC
- C23: device resistor:C-EUC0603 -> resistor:C-EUC0402
Connections:
- new net IO10_NC2: IC3.NC-3, NC10.NC
- new net IO9_NC3: IC3.NC-2, NC9.NC
- new net IO9_NC6: IC3.NC-1, NC11.NC
- new net IO9_NC7: IC3.NC-5, NC12.NC
- new net IO9_NC8: IC3.NC-4, NC15.NC
- new net N$60: C18.1, IC3.SETC
- new net N$62: C18.2, IC3.SETP
- new net N$66: C19.1, IC3.C1
- new net QMC5883-INTERRUPT: IC3.DRDY, JP11.1
- net +3V3: now also C20.1, C21.1, IC3.S1, IC3.VDD, IC3.VDDIO
- net GND: now also C19.2, C20.2, C21.2, IC3.GND
- net SCL: now also IC3.SCL
- net SDA: now also IC3.SDA
Other:
- note added: "Released under the Creative Commons Attribution-ShareAlike 4.0 License https://creativecommons.org/licenses/by-sa/4.0/ Designed by: Tom Vavrinec RB3202S-SchoolBot https://github.com/XY"
- note removed: "Released under the Creative Commons Attribution-ShareAlike 4.0 License https://creativecommons.org/licenses/by-sa/4.0/ Designed by: Tom Vavrinec RB3202-SchoolBot https://github.com/XY"
- moved on the sheet: C3, C4, C5, C8, IM6, JP1, JP12, JP2, JP3, JP4, JP5, JP6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
