File: RB3202S/hardware/SchoolBoard.brd (EAGLE design)
At the start: 101.6 x 61 mm, 89 parts, among them IC3 QMC5883L-TR, Q1 AO3401ASOP-8_EP_5.0X5.0X1.27P, Q3 AO3401ASOP-8_EP_5.0X5.0X1.27P, SW0 TL3342F160QG/TR, SW1 TL3342F160QG/TR, SW2 TL3342F160QG/TR, SW3 TL3342F160QG/TR, U1 MPU-6050, X1 POWER_IN, X2 POWER_IN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

Commit message: commit
Parts:
- added C69, C70: 10uf, rcl:C0402K
- added JP13: (no value), pinhead:1X04
- added MAX1: MAX485, maxim:SO08
- added Q10: (no value), transistors:SOT23
- added R48: 120, rcl:R0402
- added R49, R50: 20k, rcl:R0402
- added R51: 10k, rcl:R0402
- added R52: 100k, rcl:R0402
- added SJ1: (no value), jumper:SJ
- U$9: value DRV8833HTSSOP -> DRV8833CPWPR; device texas-cc2541:HTSSOP -> DRV8833CPWPR:SOP65P640X120-17N
- moved C19 2.54 mm to (33.8, 29.2)
- moved IC3 2.54 mm to (30.5, 30.5)
- moved C18 2.54 mm to (35.6, 30.0)
- moved JP11 2.54 mm to (30.2, 34.0)
- moved C20 2.54 mm to (31.2, 27.9)
- moved U$9 0.63 mm to (75.4, 38.7)
Connections:
- new net A: JP13.2, MAX1.6, R48.2, R50.1
- new net B: JP13.3, MAX1.7, R49.1, SJ1.2
- new net N$6: R48.1, SJ1.1
- new net RX-485-5V: MAX1.1, Q10.3
- net +3V3: now also IC3.S1, Q10.1, R51.2; no longer IC3.4
- net +5V: now also C69.1, C70.1, JP13.4, MAX1.8, R49.2
- net GND: now also C69.2, C70.2, JP13.1, MAX1.5, R50.2, R52.2, U$9.13, U$9.17, U$9.3, U$9.6; no longer U$9.AISEN, U$9.BISEN, U$9.GND
- net GPIO21: now also MAX1.2, MAX1.3, R52.1
- net GPIO36: now also MAX1.4
- net GPIO39: now also Q10.2, R51.1
- net IO9_NC2: now also U$9.8; no longer U$9.NFAULT
- net M1A: now also U$9.2; no longer U$9.AOUT1
- net M1B: now also U$9.4; no longer U$9.AOUT2
- net M2A: now also U$9.7; no longer U$9.BOUT1
- net M2B: now also U$9.5; no longer U$9.BOUT2
- net N$23: now also U$9.14; no longer U$9.VINT
- net N$25: now also U$9.11; no longer U$9.VCP
- net PWM_A0: now also U$9.16; no longer U$9.AIN1
- net PWM_A1: now also U$9.15; no longer U$9.AIN2
- net PWM_B0: now also U$9.9; no longer U$9.BIN1
- net PWM_B1: now also U$9.10; no longer U$9.BIN2
- net SLEEP: now also U$9.1; no longer U$9.NSLEEP
- net VCC: now also U$9.12; no longer U$9.VM
Routing:
- net +5V: track 101.0 -> 150.4 mm, vias 0 -> 4
- net GPIO36: track 58.4 -> 98.8 mm, vias 0 -> 3
- net GPIO21: track 93.2 -> 130.6 mm
- net B: track 0.00 -> 32.4 mm
- net GPIO39: track 56.0 -> 83.6 mm, vias 0 -> 1
- net A: track 0.00 -> 23.2 mm
- net +3V3: track 158.2 -> 180.7 mm
- net GND: track 9.34 -> 1.19 mm, vias 52 -> 63
- net RX-485-5V: track 0.00 -> 5.44 mm
- net N$6: track 0.00 -> 3.90 mm
- net SCL: track 116.5 -> 114.1 mm
- net SDA: track 122.3 -> 119.9 mm
- net PWM_B0: track 44.4 -> 43.0 mm
- net VCC: track 84.6 -> 85.6 mm
- net PWM_B1: track 42.8 -> 42.1 mm
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