File: RB3202S/hardware/SchoolBoard.sch (EAGLE design)
At the start: 104 parts, among them IC3 QMC5883L-TR, Q1 AO3401ASOP-8_EP_5.0X5.0X1.27P, Q3 AO3401ASOP-8_EP_5.0X5.0X1.27P, SW0 TL3342F160QG/TR, SW1 TL3342F160QG/TR, SW2 TL3342F160QG/TR, SW3 TL3342F160QG/TR, U1 MPU-6050, X1 POWER_IN, X2 POWER_IN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

Commit message: commit
Parts:
- added C69, C70: 10uf, rcl:C-EUC0402K
- added JP13: (no value), pinhead:PINHD-1X4
- added MAX1: MAX485, maxim:MAX485
- added Q10: (no value), transistors:N-MOSFET-SOT23-GSD
- added R48: 120, rcl:R-EU_R0402
- added R49, R50: 20k, rcl:R-EU_R0402
- added R51: 10k, rcl:R-EU_R0402
- added R52: 100k, rcl:R-EU_R0402
- added SJ1: (no value), jumper:SJ
- U$9: value DRV8833HTSSOP -> DRV8833CPWPR; device texas-cc2541:DRV8833HTSSOP -> DRV8833CPWPR:DRV8833CPWPR
Connections:
- new net A: JP13.2, MAX1.A, R48.2, R50.1
- new net B: JP13.3, MAX1.B, R49.1, SJ1.2
- new net N$6: R48.1, SJ1.1
- new net RX-485-5V: MAX1.RO, Q10.D
- net +3V3: now also Q10.G, R51.2
- net +5V: now also C69.1, C70.1, JP13.4, MAX1.VCC, R49.2
- net GND: now also C69.2, C70.2, JP13.1, MAX1.GND, R50.2, R52.2
- net GPIO21: now also MAX1.DE, MAX1.RE/, R52.1
- net GPIO36: now also MAX1.DI
- net GPIO39: now also Q10.S, R51.1
- net M1B: now also U$9.AOUT2; no longer U$9.AUOT2
- net N$62: now also IC3.STEP; no longer IC3.SETP
Other:
- note added: "5V-PIN"
- note added: "BAT-REF"
- note added: "I-SERVA"
- note added: "LED"
- note added: "SWX"
- note removed: "AD1"
- note removed: "rezerve_AD1"

Commit message: loga
Parts:
- C69, C70: device rcl:C-EUC0402K -> rcl:C-EUC0805
Changed lines of the file:
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@@
 <part name="P+129" library="supply1" library_urn="urn:adsk.eagle:library:371" deviceset="+5V" device=""/>
 <part name="GND144" library="supply1" library_urn="urn:adsk.eagle:library:371" deviceset="GND" device=""/>
-<part name="C69" library="rcl" library_urn="urn:adsk.eagle:library:334" deviceset="C-EU" device="C0402K" package3d_urn="urn:adsk.eagle:package:23679/2" value="10uf"/>
-<part name="C70" library="rcl" library_urn="urn:adsk.eagle:library:334" deviceset="C-EU" device="C0402K" package3d_urn="urn:adsk.eagle:package:23679/2" value="10uf"/>
+<part name="C69" library="rcl" library_urn="urn:adsk.eagle:library:334" deviceset="C-EU" device="C0805" package3d_urn="urn:adsk.eagle:package:23617/2" value="10uf"/>
+<part name="C70" library="rcl" library_urn="urn:adsk.eagle:library:334" deviceset="C-EU" device="C0805" package3d_urn="urn:adsk.eagle:package:23617/2" value="10uf"/>
 <part name="P+134" library="supply1" library_urn="urn:adsk.eagle:library:371" deviceset="+5V" device=""/>
 <part name="P+135" library="supply1" library_urn="urn:adsk.eagle:library:371" deviceset="+5V" device=""/>
