File: RB3202S/hardware/V0.1/SchoolBoard.brd (EAGLE design)
At the start: 101.6 x 61 mm, 100 parts, among them IC3 QMC5883L-TR, Q1 AO3401ASOP-8_EP_5.0X5.0X1.27P, Q3 AO3401ASOP-8_EP_5.0X5.0X1.27P, SW0 TL3342F160QG/TR, SW1 TL3342F160QG/TR, SW2 TL3342F160QG/TR, SW3 TL3342F160QG/TR, U1 MPU-6050, X1 POWER_IN, X2 POWER_IN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

Commit message: BlackBox standard
Other:
- board text added: "C:/Users/Tomas_Vavrinec/Desktop/83230147_1110853902579322_2686908253064921088_n.bmp"
- board text removed: "JESPER RB3202S_V1.0"
